File: Adafruit-nRF52-Bluefruit-Feather-PCB-master/Adafruit nRF52840 Bluefruit Feather Express Rev D/Adafruit nRF52840 Bluefruit Feather Express Rev D.kicad_pcb (KiCad board)
At the start: 4 copper layers, 333.6 x 124 mm, 380 parts, among them IC2 GD25Q16, J1 USB_C_Receptacle_USB2.0, Q3 DMG2305, SW101 KMR2, SW102 KMR2, U2 AP2112(3.3V), U3 MCP73831T-2ACI/OT, X3 JSTPH, Y2 32.768

Commit message: work
Parts:
- removed the D10 at (269.1, 51.4)
- removed the D11 at (288.2, 51.4)
- removed the D12 at (307.2, 51.4)
- removed the D13 at (326.3, 51.4)
- removed the D14 at (350.1, 51.4)
- removed the D15 at (369.1, 51.4)
- removed the D2 at (97.7, 51.4)
- removed the D3 at (116.7, 51.4)
- removed the D4 at (135.8, 51.4)
- removed the D5 at (154.8, 51.4)
- removed the D6 at (183.4, 51.4)
- removed the D7 at (202.4, 51.4)
- removed the D8 at (221.5, 51.4)
- removed the D9 at (240.5, 51.4)
- removed FID1, FID2: FIDUCIAL_1MM, Adafruit nRF52840 Bluefruit Feather Express Rev D:FIDUCIAL_1MM
- added R7: 100k, Resistor_SMD:R_0603_1608Metric, B.Cu at (68.7, 58.3)
- added R8: 100k, Resistor_SMD:R_0603_1608Metric, B.Cu at (63.2, 58.3)
- added R9: 100k, Resistor_SMD:R_0603_1608Metric, B.Cu at (194.3, 153.3)
- added U1: USBLC6-2SC6, Package_TO_SOT_SMD:SOT-23-6, B.Cu at (73.4, 50.5)
- R12: value 100K -> 100k; footprint Adafruit nRF52840 Bluefruit Feather Express Rev D:RESPACK_4X0603 -> Resistor_SMD:R_0603_1608Metric
- moved D104 179.1 mm to (197.8, 168.7)
- moved D102 178.1 mm to (200.7, 168.9)
- moved R2 170.4 mm to (201.9, 172.5)
- moved R5 170.4 mm to (197.9, 165.0)
- moved D103 161.3 mm to (85.2, 37.9), turned to 90 degrees
- moved R3 160.1 mm to (89.2, 37.9), turned to 0 degrees
- moved R4 150.8 mm to (83.7, 50.9), turned to -90 degrees
- moved U3 150.4 mm to (80.0, 50.9)
- moved C9 149.5 mm to (76.9, 53.3), turned to 90 degrees
- moved R12 140.5 mm to (194.3, 149.0), turned to -90 degrees
- moved TP1 117.2 mm to (156.2, 143.1)
- moved SW102 34.6 mm to (163.5, 181.6)
- moved SW101 34.6 mm to (163.5, 177.4)
- moved C10 31.0 mm to (144.8, 180.0)
- moved C3 31.0 mm to (144.8, 175.0)
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Connections:
- MDBT1 pad 34: /USBD- -> Net-(MDBT1-D-)
- MDBT1 pad 35: /USBD+ -> Net-(MDBT1-D+)
- R10 pad 1: Net-(D-0-PadTP) -> /USBD+
- R10 pad 2: /USBD+ -> Net-(MDBT1-D+)
- R11 pad 1: Net-(D+0-PadTP) -> /USBD-
- R11 pad 2: /USBD- -> Net-(MDBT1-D-)
- R12 pad 1: VBUS -> VBAT
- R12 pad 2: /EN -> /VDIV
Routing:
- net VBAT: track 0.00 -> 360.3 mm
- net /USBD+: track 0.00 -> 151.3 mm, vias 0 -> 2
- net /USBD-: track 0.00 -> 150.7 mm, vias 0 -> 2
- net VBUS: track 0.00 -> 48.2 mm, vias 0 -> 3
- net Net-(D1-A): track 0.00 -> 20.6 mm
- net Net-(U3-STAT): track 0.00 -> 19.6 mm
- net Net-(Q3-S): track 0.00 -> 18.6 mm
- net Net-(D-0-PadTP): track 0.00 -> 15.6 mm, vias 0 -> 2
- net Net-(D+0-PadTP): track 0.00 -> 15.4 mm, vias 0 -> 2
- net Net-(J1-CC2): track 0.00 -> 12.7 mm
- net Net-(J1-CC1): track 0.00 -> 12.7 mm
- net /EN: track 0.00 -> 10.5 mm
- net /QSPI_DATA2: track 0.00 -> 7.06 mm, vias 0 -> 2
- net Net-(MDBT1-P0.01/XL2): track 0.00 -> 7.05 mm
- net Net-(MDBT1-P0.00/XL1): track 0.00 -> 7.03 mm
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