File: Adafruit-nRF52-Bluefruit-Feather-PCB-master/Adafruit nRF52840 Bluefruit Feather Express Rev D/Adafruit nRF52840 Bluefruit Feather Express Rev D.kicad_sch (KiCad schematic)
At the start: 39 parts, among them IC2 GD25Q16, J1 USB_C_Receptacle_USB2.0, Q3 DMG2305, SW101 KMR2, SW102 KMR2, U2 AP2112(3.3V), U3 MCP73831T-2ACI/OT, X3 JSTPH, Y2 32.768

Commit message: work
Parts:
- removed FID1, FID2: FIDUCIAL_1MM, Adafruit nRF52840 Bluefruit Feather Express Rev D:FIDUCIAL_1MM, symbol Adafruit nRF52840 Bluefruit Feather Express Rev D-eagle-import:FIDUCIAL_1MM
- removed R12: 100K, Adafruit nRF52840 Bluefruit Feather Express Rev D:RESPACK_4X0603, symbol Adafruit nRF52840 Bluefruit Feather Express Rev D-eagle-import:RESISTOR_4PACK
- added R12, R7, R8, R9: 100k, Resistor_SMD:R_0603_1608Metric, symbol Device:R
- added U0: USBLC6-2SC6, Package_TO_SOT_SMD:SOT-23-6, symbol Power_Protection:USBLC6-2SC6
Connections:
- net EN: now also R8.2
- net GND: now also R7.2, R9.2, U0.2 (GND)
- net USBD+: now also R10.1, U0.6 (I/O1); no longer MDBT1.35 (D+), R10.2
- net USBD-: now also R11.1, U0.4 (I/O2); no longer MDBT1.34 (D-), R11.2
- net VBAT: now also R12.1
- net VBUS: now also R7.1, U0.5 (VBUS)
- net VDIV: now also R12.2, R9.1
- net at C7.2, D101.C, Q3.2 (S)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: now also R8.1
- net at D+0.TP, J1.A7 (D-), J1.B7 (D-): now also U0.3 (I/O2); no longer R11.1
- net at D-0.TP, J1.A6 (D+), J1.B6 (D+): now also U0.1 (I/O1); no longer R10.1
- new net: MDBT1.34 (D-), R11.2
- new net: MDBT1.35 (D+), R10.2
Other:
- note removed: "NEOPIXEL"
- moved on the sheet: D+0, D-0
