File: Adafruit nRF52840 Bluefruit Feather Express Rev D.kicad_pcb (KiCad board)
At the start: 4 copper layers, 333.6 x 124 mm, 368 parts, among them IC2 GD25Q16, J1 USB_C_Receptacle_USB2.0, Q3 DMG2305, SW101 KMR2, SW102 KMR2, U1 USBLC6-2SC6, U2 AP2112(3.3V), U3 MCP73831T-2ACI/OT, X3 JSTPH, Y2 32.768

Commit message: Add plates
Parts:
- moved D65 1.25 mm to (159.6, 132.3), turned to 90 degrees
Changed lines of the file:
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@@
   )
   (footprint "Diode_SMD:D_SOD-323_HandSoldering" (layer "B.Cu")
-    (at 158.3255 132.316 180)
+    (at 159.5755 132.316 90)
     (descr "SOD-323")
     (tags "SOD-323")
@@
     (property "ki_keywords" "diode")
     (attr smd)
-    (fp_text reference "D65" (at 0 1.85) (layer "B.SilkS")
+    (fp_text reference "D65" (at 0 1.85 90) (layer "B.SilkS")
         (effects (font (size 1 1) (thickness 0.15)) (justify mirror))
     )
-    (fp_text value "D" (at 0.1 -1.9) (layer "B.Fab")
+    (fp_text value "D" (at 0.1 -1.9 90) (layer "B.Fab")
         (effects (font (size 1 1) (thickness 0.15)) (justify mirror))
     )
-    (fp_text user "${REFERENCE}" (at 0 1.85) (layer "B.Fab")
+    (fp_text user "${REFERENCE}" (at 0 1.85 90) (layer "B.Fab")
         (effects (font (size 1 1) (thickness 0.15)) (justify mirror))
     )
@@
     (fp_line (start 0.9 0.7) (end 0.9 -0.7)
       (stroke (width 0.1) (type solid)) (layer "B.Fab"))
-    (pad "1" smd roundrect (at -1.25 0 180) (size 1 1) (layers "B.Cu" "B.Paste" "B.Mask") (roundrect_rratio 0.25)
+    (pad "1" smd roundrect (at -1.25 0 90) (size 1 1) (layers "B.Cu" "B.Paste" "B.Mask") (roundrect_rratio 0.25)
       (net 80 "Net-(D20-K)") (pinfunction "K") (pintype "passive"))
-    (pad "2" smd roundrect (at 1.25 0 180) (size 1 1) (layers "B.Cu" "B.Paste" "B.Mask") (roundrect_rratio 0.25)
+    (pad "2" smd roundrect (at 1.25 0 90) (size 1 1) (layers "B.Cu" "B.Paste" "B.Mask") (roundrect_rratio 0.25)
       (net 152 "Net-(D65-A)") (pinfunction "A") (pintype "passive"))
     (model "${KICAD6_3DMODEL_DIR}/Diode_SMD.3dshapes/D_SOD-323.wrl"
@@
     )
   )
+  (gr_rect (start 42.5 36.3) (end 376 160.3)
+    (stroke (width 0.1) (type default)) (fill none) (layer "Eco2.User"))
   (gr_line (start 42.483 160.336) (end 42.483 36.3235)
     (stroke (width 0.1) (type default)) (layer "Edge.Cuts"))
