File: Adafruit nRF52840 Bluefruit Feather Express Rev D.kicad_pcb (KiCad board)
At the start: 4 copper layers, 333.6 x 124 mm, 368 parts, among them IC2 GD25Q16, J1 USB_C_Receptacle_USB2.0, Q3 DMG2305, SW101 KMR2, SW102 KMR2, U1 USBLC6-2SC6, U2 AP2112(3.3V), U3 MCP73831T-2ACI/OT, X3 JSTPH, Y2 32.768

Commit message: Small work
Parts:
- removed D+0, D-0: TPTP10R, Adafruit nRF52840 Bluefruit Feather Express Rev D:TP10R
- removed R1, R6: 5.1k, Resistor_SMD:R_0603_1608Metric
- removed U1: USBLC6-2SC6, Package_TO_SOT_SMD:SOT-23-6
- J1: value USB_C_Receptacle_USB2.0 -> 781710004; footprint JohnDeereLibrary:GCT USB4510-03-1-A -> footprints:CON_781710004
- moved J1 164.8 mm to (200.1, 143.3)
Routing:
- net /USBD-: track 150.7 -> 2.42 mm, vias 2 -> 1
- net /USBD+: track 151.3 -> 3.76 mm, vias 2 -> 1
- net VBUS: track 48.2 -> 27.4 mm, vias 3 -> 1
- net (no net): track 0.00 -> 19.1 mm
- net Net-(D-0-PadTP): track 15.6 -> 0.00 mm, vias 2 -> 0
- net Net-(D+0-PadTP): track 15.4 -> 0.00 mm, vias 2 -> 0
- net Net-(J1-CC2): track 12.7 -> 0.00 mm
- net Net-(J1-CC1): track 12.7 -> 0.00 mm
- net GND: track 0.35 -> 0.00 mm, vias 1 -> 0

Commit message: removed bad diodes
TODO: rotate good diodes
Parts:
- removed the D16 at (59.6, 75.2)
- removed the D17 at (78.6, 75.2)
- removed the D18 at (97.7, 75.2)
- removed the D19 at (116.7, 75.2)
- removed the D20 at (135.8, 75.2)
- removed the D21 at (154.8, 75.2)
- removed the D22 at (173.9, 75.2)
- removed the D23 at (192.9, 75.2)
- removed the D24 at (212.0, 75.2)
- removed the D25 at (231.0, 75.2)
- removed the D26 at (250.1, 75.2)
- removed the D27 at (269.1, 75.2)
- removed the D28 at (288.2, 75.2)
- removed the D29 at (316.7, 75.2)
- removed the D30 at (350.1, 75.2)
- removed the D31 at (369.1, 75.2)
- removed the D32 at (64.3, 94.2)
- removed the D33 at (88.1, 94.2)
- removed the D34 at (107.2, 94.2)
- removed the D35 at (126.2, 94.2)
- removed the D36 at (145.3, 94.2)
- removed the D37 at (164.3, 94.2)
- removed the D38 at (183.4, 94.2)
- removed the D39 at (202.4, 94.2)
- removed the D40 at (221.5, 94.2)
- removed the D41 at (240.5, 94.2)
- removed the D42 at (259.6, 94.2)
- removed the D43 at (278.6, 94.2)
- removed the D44 at (297.7, 94.2)
- removed the D45 at (321.5, 94.2)
- removed the D46 at (350.1, 94.2)
- removed the D47 at (369.1, 94.2)
- removed the D48 at (66.7, 113.3)
- removed the D49 at (92.9, 113.3)
- removed the D50 at (112.0, 113.3)
- removed the D51 at (131.0, 113.3)
- removed the D52 at (150.1, 113.3)
- removed the D53 at (169.1, 113.3)
- removed the D54 at (188.2, 113.3)
- removed the D55 at (207.2, 113.3)
- removed the D56 at (226.3, 113.3)
- removed the D57 at (245.3, 113.3)
- removed the D58 at (264.4, 113.3)
- removed the D59 at (283.4, 113.3)
- removed the D60 at (314.4, 113.3)
- removed the D61 at (71.5, 132.3)
- removed the D62 at (102.4, 132.3)
- removed the D63 at (121.5, 132.3)
- removed the D64 at (140.5, 132.3)
- removed the D65 at (159.6, 132.3)
- removed the D66 at (178.6, 132.3)
- removed the D67 at (197.7, 132.3)
- removed the D68 at (216.7, 132.3)
- removed the D69 at (235.8, 132.3)
- removed the D70 at (254.8, 132.3)
- removed the D71 at (273.9, 132.3)
- removed the D72 at (309.6, 132.3)
- removed the D73 at (350.1, 132.3)
- removed the D74 at (61.9, 151.4)
- removed the D75 at (85.8, 151.4)
- removed the D76 at (109.6, 151.4)
- removed the D77 at (181.0, 151.4)
- removed the D78 at (252.4, 151.4)
- removed the D79 at (276.3, 151.4)
- removed the D80 at (300.1, 151.4)
- removed the D81 at (331.0, 151.4)
- removed the D82 at (350.1, 151.4)
- removed the D83 at (369.1, 151.4)
- moved D103 323.1 mm to (388.7, 148.8)
- moved R3 323.1 mm to (392.6, 148.8)
- moved C9 314.8 mm to (379.9, 138.8)
- moved U3 314.8 mm to (382.9, 136.4)
- moved R4 313.5 mm to (380.6, 151.3)
- moved R9 134.9 mm to (95.2, 61.7)
- moved R12 134.5 mm to (95.2, 58.1)
- moved MDBT1 133.0 mm to (75.3, 44.1), turned to 180 degrees
- moved R10 132.5 mm to (19.9, 110.0)
- moved R11 132.5 mm to (18.0, 110.0)
- moved L1 130.4 mm to (20.7, 102.2)
- moved IC2 129.2 mm to (67.1, 45.9), turned to -90 degrees
- moved Y2 119.0 mm to (78.1, 54.7), turned to 0 degrees
- moved J1 116.8 mm to (119.7, 58.7), turned to -90 degrees
- moved C1 113.7 mm to (79.3, 58.9), turned to -90 degrees
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Routing:
- net VBAT: track 360.3 -> 130.7 mm
- net /VDIV: track 0.00 -> 25.4 mm
- net Net-(U3-STAT): track 19.6 -> 0.00 mm
- net (no net): track 19.1 -> 0.00 mm
- net VBUS: track 27.4 -> 9.45 mm, vias 1 -> 0
- net /EN: track 10.5 -> 1.99 mm
- net Net-(Q3-S): track 18.6 -> 12.9 mm
- net 3.3V: track 3.56 -> 7.89 mm
- net Net-(U3-PROG): track 2.94 -> 0.00 mm
- net Net-(D103-PadC): track 2.07 -> 0.00 mm
Other:
- outline, holes or cut-outs redrawn
- board text added: "350mAh #2750"

Commit message: work on matrix
Parts:
- removed the REF** at (61.6, 110.2)
- removed the REF** at (304.5, 129.3)
- removed the REF** at (309.3, 110.2)
- removed the REF** at (175.9, 148.3)
- removed the REF** at (66.4, 129.3)
- moved D60 1.09 mm to (315.0, 114.2), turned to 90 degrees
- moved D71 1.09 mm to (274.5, 133.2), turned to 90 degrees
- moved D72 1.09 mm to (310.2, 133.2), turned to 90 degrees
- moved D73 1.09 mm to (350.7, 133.2), turned to 90 degrees
- moved D82 1.09 mm to (350.7, 152.2), turned to 90 degrees
- moved D83 1.09 mm to (369.8, 152.2), turned to 90 degrees
- moved D48 1.09 mm to (67.3, 114.2), turned to 90 degrees
- moved D49 1.09 mm to (93.5, 114.2), turned to 90 degrees
- moved D51 1.09 mm to (131.6, 114.2), turned to 90 degrees
- moved D52 1.09 mm to (150.7, 114.2), turned to 90 degrees
- moved D54 1.09 mm to (188.8, 114.2), turned to 90 degrees
- moved D55 1.09 mm to (207.8, 114.2), turned to 90 degrees
- moved D56 1.09 mm to (226.9, 114.2), turned to 90 degrees
- moved D57 1.09 mm to (245.9, 114.2), turned to 90 degrees
- moved D50 1.09 mm to (112.6, 114.2), turned to 90 degrees
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Connections:
- D73 pad 2: unconnected-(D73-A-Pad2) -> Net-(D73-A)
- SW73 pad 2: unconnected-(SW73-Pad2) -> Net-(D73-A)
Routing:
- net Net-(SW16-Pad1): track 0.00 -> 347.5 mm
- net Net-(SW32-Pad1): track 0.00 -> 342.7 mm
- net Net-(SW74-Pad1): track 0.00 -> 331.5 mm
- net Net-(SW61-Pad1): track 0.00 -> 309.9 mm
- net Net-(SW1-Pad1): track 0.00 -> 304.3 mm
- net Net-(SW48-Pad1): track 0.00 -> 280.2 mm
- net VBAT: track 130.7 -> 22.5 mm
- net Net-(SW77B-DO): track 0.00 -> 67.1 mm
- net Net-(SW76B-DO): track 0.00 -> 67.1 mm
- net Net-(SW72B-DO): track 0.00 -> 36.1 mm
- net Net-(SW71B-DO): track 0.00 -> 31.4 mm
- net Net-(SW61B-DO): track 0.00 -> 26.8 mm
- net Net-(SW80B-DO): track 0.00 -> 26.6 mm
- net Net-(D9-A): track 0.00 -> 21.3 mm
- net Net-(D20-A): track 0.00 -> 21.1 mm
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
Commit message: small work done
Parts:
- removed the REF** at (61.6, 110.2)
- removed the REF** at (66.4, 129.3)
- added REF**: gateron-ks27-6-25U, fingerpunch:gateron-ks27-6-25U, F.Cu at (175.9, 148.3)
- added gateron_stabs: gateron-ks57-2U, fingerpunch:gateron-ks57-2U, F.Cu at (61.6, 110.2)
- added gateron_stabs: gateron-ks57-2U, fingerpunch:gateron-ks57-2U, F.Cu at (66.4, 129.3)
- moved D103 266.9 mm to (151.9, 25.6)
- moved R3 266.9 mm to (155.8, 25.6)
- moved R4 266.9 mm to (143.8, 28.1)
- moved C9 266.9 mm to (143.1, 15.6)
- moved U3 266.9 mm to (146.1, 13.2)
- moved C10 170.5 mm to (97.6, 16.2)
- moved C5 170.5 mm to (91.4, 12.3)
- moved C6 170.5 mm to (91.4, 14.8)
- moved D102 170.5 mm to (134.7, 18.6)
- moved R5 170.5 mm to (133.5, 14.1)
- moved SW102 170.5 mm to (116.4, 17.8)
- moved TP1 170.5 mm to (104.7, 2.48)
- moved C3 170.5 mm to (97.6, 11.2)
- moved C4 170.5 mm to (97.6, 13.7)
- moved D104 170.5 mm to (131.8, 18.4)
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Routing:
- net Net-(SW29B-DO): track 0.00 -> 28.8 mm
- net Net-(SW59B-DO): track 0.00 -> 26.6 mm
- net Net-(SW10B-DI): track 0.00 -> 24.2 mm
- net Net-(SW5B-DO): track 0.00 -> 24.2 mm
- net Net-(SW45B-DO): track 0.00 -> 24.1 mm
- net Net-(SW28B-DO): track 0.00 -> 24.0 mm
- net Net-(SW48B-DO): track 0.00 -> 22.4 mm
- net Net-(SW13B-DO): track 0.00 -> 19.4 mm
- net Net-(SW44B-DO): track 0.00 -> 19.3 mm
- net Net-(SW32B-DO): track 0.00 -> 19.3 mm
- net Net-(SW51B-DO): track 0.00 -> 14.7 mm
- net Net-(SW50B-DO): track 0.00 -> 14.7 mm
- net Net-(SW49B-DO): track 0.00 -> 14.7 mm
- net Net-(SW56B-DO): track 0.00 -> 14.7 mm
- net Net-(SW54B-DO): track 0.00 -> 14.7 mm
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