File: Keyboard_Matrix.kicad_sch (KiCad schematic)
At the start: 249 parts

Commit message: work on matrix
Connections:
- net at D73.2 (A): now also SW73.2
Other:
- moved on the sheet: SW73A
Changed lines of the file:
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@@
     (stroke (width 0) (type default))
   )
-  (wire (pts (xy 270.51 82.55) (xy 290.83 82.55))
+  (wire (pts (xy 270.51 82.55) (xy 289.56 82.55))
     (stroke (width 0) (type default))
   )
@@
     )
   )
-  (symbol (lib_id "JohnDeere:MX_NEO") (at 293.37 85.09 0) (unit 1)
+  (symbol (lib_id "JohnDeere:MX_NEO") (at 292.1 85.09 0) (unit 1)
     (in_bom yes) (on_board yes) (dnp no) (fields_autoplaced)
-    (property "Reference" "SW73" (at 293.37 81.28 0)
+    (property "Reference" "SW73" (at 292.1 81.28 0)
       (effects (font (size 1.27 1.27)))
     )
-    (property "Value" "~" (at 293.37 80.01 0)
+    (property "Value" "~" (at 292.1 80.01 0)
       (effects (font (size 1.27 1.27)))
     )
-    (property "Footprint" "fingerpunch:gateron-ks27-choc-v1-mx-hotswap" (at 293.37 80.01 0)
+    (property "Footprint" "fingerpunch:gateron-ks27-choc-v1-mx-hotswap" (at 292.1 80.01 0)
       (effects (font (size 1.27 1.27)) hide)
     )
-    (property "Datasheet" "" (at 293.37 80.01 0)
+    (property "Datasheet" "" (at 292.1 80.01 0)
       (effects (font (size 1.27 1.27)) hide)
     )
