File: Plate/Every83_Plate.kicad_pcb (KiCad board)
At the start: 4 copper layers, 333.6 x 134 mm, 84 parts

Commit message: WIP
Parts:
- removed REF**: STAB_choc_6.25u, marbastlib-xp-choc:STAB_choc_6.25u
- SW77: footprint JohnDeereLibrary:Gateron KS33 Plate -> JohnDeereLibrary:Gateron Low Profile Stabilizer Plate Cutout 6.25u
Other:
- outline, holes or cut-outs redrawn
- copper layers 4 -> 2
