File: Plate/Keyboard_Matrix.kicad_sch (KiCad schematic)
At the start: 83 parts

Commit message: WIP
Parts:
- SW77: footprint JohnDeereLibrary:Gateron KS33 Plate -> JohnDeereLibrary:Gateron Low Profile Stabilizer Plate Cutout 6.25u
Changed lines of the file:
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@@
       (effects (font (size 1.27 1.27)))
     )
-    (property "Footprint" "JohnDeereLibrary:Gateron KS33 Plate" (at 121.92 99.06 0)
+    (property "Footprint" "JohnDeereLibrary:Gateron Low Profile Stabilizer Plate Cutout 6.25u" (at 121.92 99.06 0)
       (effects (font (size 1.27 1.27)) hide)
     )
@@
       (effects (font (size 1.27 1.27)))
     )
-    (property "Footprint" "JohnDeereLibrary:Gateron KS33 Plate" (at 148.59 342.9 0)
-      (effects (font (size 1.27 1.27)) hide)
-    )
+    (property "Footprint" "JohnDeereLibrary:Gateron Low Profile Stabilizer Plate Cutout 6.25u" (at 148.59 342.9 0)
+      (effects (font (size 1.27 1.27)) hide)
+    )
