File: PCB/_autosave-Every83_PCB.kicad_sch (KiCad schematic)
At the start: 29 parts, among them J1 781710004, J2 Conn_01x08_Socket, J3 SM03B-SRSS-TB, J4 SM03B-SRSS-TB, J5 Conn_01x08_Socket, J6 Conn_01x03_Socket, J7 Conn_01x02_Socket, Q3 DMG2305, SW101 KMR2, SW102 KMR2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

Commit message: small changes
Other:
- removed sheet Power Daughter Board
Changed lines of the file:
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@@
-		)
-	)
-	(sheet
-		(at 274.32 80.01)
-		(size 20.32 29.21)
-		(fields_autoplaced yes)
-		(stroke
-			(width 0.1524)
-			(type solid)
-		)
-		(fill
-			(color 0 0 0 0.0000)
-		)
-		(property "Sheetname" "Power Daughter Board"
-			(at 274.32 79.2984 0)
-			(effects
-				(font
-					(size 1.27 1.27)
-				)
-				(justify left bottom)
-			)
-		)
-		(property "Sheetfile" "Power_Daughterboard.kicad_sch"
-			(at 274.32 109.8046 0)
-			(effects
-				(font
-					(size 1.27 1.27)
-				)
-				(justify left top)
-			)
-		)
-		(instances
-			(project "Every83_PCB"
-				(path "/ea2432c4-eb7a-431a-b465-8c00cfcb4450"
-					(page "3")
-				)
-			)
 		)
 	)
