File: PCB/Every83_PCB.kicad_pcb (KiCad board)
At the start: 4 copper layers, 330.2 x 118.6 mm, 290 parts, among them J1 781710004, J10 Conn_01x01, J11 Conn_01x05_Pin, J2 Conn_01x08_Socket, J5 Conn_01x08_Socket, J6 Conn_01x02_Pin, J7 Conn_02x03_Counter_Clockwise, Q1 MMDT2222A, Q3 DMG2305, SW101 KMR2, SW102 KMR2, U1 Core52840, U2 AP2112(3.3V), U3 MCP73831T-2ACI/OT

Commit message: update neopixel power plane
Parts:
- removed J11: Conn_01x05_Pin, Connector_PinHeader_1.27mm:PinHeader_1x05_P1.27mm_Vertical
- added Q2: 2N7002, Package_TO_SOT_SMD:SOT-23, B.Cu at (174.5, 173.9)
- added Q4: AO3401A, Package_TO_SOT_SMD:SOT-23, B.Cu at (174.5, 178.5)
- added R13: 100R, Resistor_SMD:R_0603_1608Metric, B.Cu at (170.0, 172.7)
- added R14: 10K, Resistor_SMD:R_0603_1608Metric, B.Cu at (170.0, 175.2)
- added R15: 10K, Resistor_SMD:R_0603_1608Metric, B.Cu at (170.0, 177.8)
- C11, C12, C13, C14, C15, C16, C17, C18, C19, C20, C21, C22, C23, C24, C25, C26, C27, C28, C29, C30, C31, C32, C33, C34, C35, C36, C37, C38, C39, C40, C41, C42, C43, C44, C45, C46, C47, C48, C49, C50, C51, C52, C53, C54, C55, C56, C57, C58, C59, C60, C61, C62, C63, C64, C65, C66, C67, C68, C69, C70, C71, C72, C73, C74, C75, C76, C77, C78, C79, C80, C81, C82, C83, C84, C85, C86, C87, C88, C89, C90, C91, C92, C93: value C -> 100n
- D1, D10, D11, D12, D13, D14, D15, D16, D17, D18, D19, D2, D20, D21, D22, D23, D24, D25, D26, D27, D28, D29, D3, D30, D31, D32, D33, D34, D35, D36, D37, D38, D39, D4, D40, D41, D42, D43, D44, D45, D46, D47, D48, D49, D5, D50, D51, D52, D53, D54, D55, D56, D57, D58, D59, D6, D60, D61, D62, D63, D64, D65, D66, D67, D68, D69, D7, D70, D71, D72, D73, D74, D75, D76, D77, D78, D79, D8, D80, D81, D82, D83, D9: value D -> 1n4148
- moved J2 214.6 mm to (141.5, 172.8)
- moved J5 214.6 mm to (161.1, 172.7)
- moved J1 8.71 mm to (144.2, 144.1)
- moved C3 7.17 mm to (163.3, 147.5)
- moved R7 7.17 mm to (152.3, 148.0)
- moved R8 7.17 mm to (158.4, 143.9)
- moved U2 7.17 mm to (161.5, 143.9)
- moved C7 7.17 mm to (160.2, 147.3)
- moved C8 7.17 mm to (165.0, 143.9)
- moved D101 7.17 mm to (155.6, 147.3)
- moved Q3 7.17 mm to (155.2, 144.0)
Connections:
- C11 pad 1: 3.3V -> NEOPIX_PWR
- C12 pad 1: 3.3V -> NEOPIX_PWR
- C13 pad 1: 3.3V -> NEOPIX_PWR
- C14 pad 1: 3.3V -> NEOPIX_PWR
- C15 pad 1: 3.3V -> NEOPIX_PWR
- C16 pad 1: 3.3V -> NEOPIX_PWR
- C17 pad 1: 3.3V -> NEOPIX_PWR
- C18 pad 1: 3.3V -> NEOPIX_PWR
- C19 pad 1: 3.3V -> NEOPIX_PWR
- C20 pad 1: 3.3V -> NEOPIX_PWR
- C21 pad 1: 3.3V -> NEOPIX_PWR
- C22 pad 1: 3.3V -> NEOPIX_PWR
- C23 pad 1: 3.3V -> NEOPIX_PWR
- C24 pad 1: 3.3V -> NEOPIX_PWR
- C25 pad 1: 3.3V -> NEOPIX_PWR
- C26 pad 1: 3.3V -> NEOPIX_PWR
- C27 pad 1: 3.3V -> NEOPIX_PWR
- C28 pad 1: 3.3V -> NEOPIX_PWR
- C29 pad 1: 3.3V -> NEOPIX_PWR
- C30 pad 1: 3.3V -> NEOPIX_PWR
- C31 pad 1: 3.3V -> NEOPIX_PWR
- C32 pad 1: 3.3V -> NEOPIX_PWR
- C33 pad 1: 3.3V -> NEOPIX_PWR
- C34 pad 1: 3.3V -> NEOPIX_PWR
- C35 pad 1: 3.3V -> NEOPIX_PWR
- C36 pad 1: 3.3V -> NEOPIX_PWR
- C37 pad 1: 3.3V -> NEOPIX_PWR
- C38 pad 1: 3.3V -> NEOPIX_PWR
- C39 pad 1: 3.3V -> NEOPIX_PWR
- C40 pad 1: 3.3V -> NEOPIX_PWR
- C41 pad 1: 3.3V -> NEOPIX_PWR
- C42 pad 1: 3.3V -> NEOPIX_PWR
- C43 pad 1: 3.3V -> NEOPIX_PWR
- C44 pad 1: 3.3V -> NEOPIX_PWR
- C45 pad 1: 3.3V -> NEOPIX_PWR
- C46 pad 1: 3.3V -> NEOPIX_PWR
- C47 pad 1: 3.3V -> NEOPIX_PWR
- C48 pad 1: 3.3V -> NEOPIX_PWR
- C49 pad 1: 3.3V -> NEOPIX_PWR
- C50 pad 1: 3.3V -> NEOPIX_PWR
- C51 pad 1: 3.3V -> NEOPIX_PWR
- C52 pad 1: 3.3V -> NEOPIX_PWR
- C53 pad 1: 3.3V -> NEOPIX_PWR
- C54 pad 1: 3.3V -> NEOPIX_PWR
- C55 pad 1: 3.3V -> NEOPIX_PWR
- C56 pad 1: 3.3V -> NEOPIX_PWR
- C57 pad 1: 3.3V -> NEOPIX_PWR
- C58 pad 1: 3.3V -> NEOPIX_PWR
- C59 pad 1: 3.3V -> NEOPIX_PWR
- C60 pad 1: 3.3V -> NEOPIX_PWR
- C61 pad 1: 3.3V -> NEOPIX_PWR
- C62 pad 1: 3.3V -> NEOPIX_PWR
- C63 pad 1: 3.3V -> NEOPIX_PWR
- C64 pad 1: 3.3V -> NEOPIX_PWR
- C65 pad 1: 3.3V -> NEOPIX_PWR
- C66 pad 1: 3.3V -> NEOPIX_PWR
- C67 pad 1: 3.3V -> NEOPIX_PWR
- C68 pad 1: 3.3V -> NEOPIX_PWR
- C69 pad 1: 3.3V -> NEOPIX_PWR
- C70 pad 1: 3.3V -> NEOPIX_PWR
- C71 pad 1: 3.3V -> NEOPIX_PWR
- C72 pad 1: 3.3V -> NEOPIX_PWR
- C73 pad 1: 3.3V -> NEOPIX_PWR
- C74 pad 1: 3.3V -> NEOPIX_PWR
- C75 pad 1: 3.3V -> NEOPIX_PWR
- C76 pad 1: 3.3V -> NEOPIX_PWR
- C77 pad 1: 3.3V -> NEOPIX_PWR
- C78 pad 1: 3.3V -> NEOPIX_PWR
- C79 pad 1: 3.3V -> NEOPIX_PWR
- C80 pad 1: 3.3V -> NEOPIX_PWR
- C81 pad 1: 3.3V -> NEOPIX_PWR
- C82 pad 1: 3.3V -> NEOPIX_PWR
- C83 pad 1: 3.3V -> NEOPIX_PWR
- C84 pad 1: 3.3V -> NEOPIX_PWR
- C85 pad 1: 3.3V -> NEOPIX_PWR
- C86 pad 1: 3.3V -> NEOPIX_PWR
- C87 pad 1: 3.3V -> NEOPIX_PWR
- C88 pad 1: 3.3V -> NEOPIX_PWR
- C89 pad 1: 3.3V -> NEOPIX_PWR
- C90 pad 1: 3.3V -> NEOPIX_PWR
- C91 pad 1: 3.3V -> NEOPIX_PWR
- C92 pad 1: 3.3V -> NEOPIX_PWR
- C93 pad 1: 3.3V -> NEOPIX_PWR
- J5 pad 1: 9 -> GND
- J5 pad 2: 10 -> 9
- SW1 pad 4: 3.3V -> NEOPIX_PWR
- SW10 pad 4: 3.3V -> NEOPIX_PWR
- SW11 pad 4: 3.3V -> NEOPIX_PWR
- SW12 pad 4: 3.3V -> NEOPIX_PWR
- SW13 pad 4: 3.3V -> NEOPIX_PWR
- SW14 pad 4: 3.3V -> NEOPIX_PWR
- SW15 pad 4: 3.3V -> NEOPIX_PWR
- SW16 pad 4: 3.3V -> NEOPIX_PWR
- SW17 pad 4: 3.3V -> NEOPIX_PWR
- SW18 pad 4: 3.3V -> NEOPIX_PWR
- SW19 pad 4: 3.3V -> NEOPIX_PWR
- SW2 pad 4: 3.3V -> NEOPIX_PWR
- SW20 pad 4: 3.3V -> NEOPIX_PWR
- SW21 pad 4: 3.3V -> NEOPIX_PWR
- SW22 pad 4: 3.3V -> NEOPIX_PWR
- SW23 pad 4: 3.3V -> NEOPIX_PWR
- SW24 pad 4: 3.3V -> NEOPIX_PWR
- SW25 pad 4: 3.3V -> NEOPIX_PWR
- SW26 pad 4: 3.3V -> NEOPIX_PWR
- SW27 pad 4: 3.3V -> NEOPIX_PWR
- SW28 pad 4: 3.3V -> NEOPIX_PWR
- SW29 pad 4: 3.3V -> NEOPIX_PWR
- SW3 pad 4: 3.3V -> NEOPIX_PWR
- SW30 pad 4: 3.3V -> NEOPIX_PWR
- SW31 pad 4: 3.3V -> NEOPIX_PWR
- SW32 pad 4: 3.3V -> NEOPIX_PWR
- SW33 pad 4: 3.3V -> NEOPIX_PWR
- SW34 pad 4: 3.3V -> NEOPIX_PWR
- SW35 pad 4: 3.3V -> NEOPIX_PWR
- SW36 pad 4: 3.3V -> NEOPIX_PWR
- SW37 pad 4: 3.3V -> NEOPIX_PWR
- SW38 pad 4: 3.3V -> NEOPIX_PWR
- SW39 pad 4: 3.3V -> NEOPIX_PWR
- SW4 pad 4: 3.3V -> NEOPIX_PWR
- SW40 pad 4: 3.3V -> NEOPIX_PWR
- SW41 pad 4: 3.3V -> NEOPIX_PWR
- SW42 pad 4: 3.3V -> NEOPIX_PWR
- SW43 pad 4: 3.3V -> NEOPIX_PWR
- SW44 pad 4: 3.3V -> NEOPIX_PWR
- SW45 pad 4: 3.3V -> NEOPIX_PWR
- SW46 pad 4: 3.3V -> NEOPIX_PWR
- SW47 pad 4: 3.3V -> NEOPIX_PWR
- SW48 pad 4: 3.3V -> NEOPIX_PWR
- SW49 pad 4: 3.3V -> NEOPIX_PWR
- SW5 pad 4: 3.3V -> NEOPIX_PWR
- SW50 pad 4: 3.3V -> NEOPIX_PWR
- SW51 pad 4: 3.3V -> NEOPIX_PWR
- SW52 pad 4: 3.3V -> NEOPIX_PWR
- SW53 pad 4: 3.3V -> NEOPIX_PWR
- SW54 pad 4: 3.3V -> NEOPIX_PWR
- SW55 pad 4: 3.3V -> NEOPIX_PWR
- SW56 pad 4: 3.3V -> NEOPIX_PWR
- SW57 pad 4: 3.3V -> NEOPIX_PWR
- SW58 pad 4: 3.3V -> NEOPIX_PWR
- SW59 pad 4: 3.3V -> NEOPIX_PWR
- SW6 pad 4: 3.3V -> NEOPIX_PWR
- SW60 pad 4: 3.3V -> NEOPIX_PWR
- SW61 pad 4: 3.3V -> NEOPIX_PWR
- SW62 pad 4: 3.3V -> NEOPIX_PWR
- SW63 pad 4: 3.3V -> NEOPIX_PWR
- SW64 pad 4: 3.3V -> NEOPIX_PWR
- SW65 pad 4: 3.3V -> NEOPIX_PWR
- SW66 pad 4: 3.3V -> NEOPIX_PWR
- SW67 pad 4: 3.3V -> NEOPIX_PWR
- SW68 pad 4: 3.3V -> NEOPIX_PWR
- SW69 pad 4: 3.3V -> NEOPIX_PWR
- SW7 pad 4: 3.3V -> NEOPIX_PWR
- SW70 pad 4: 3.3V -> NEOPIX_PWR
- SW71 pad 4: 3.3V -> NEOPIX_PWR
- SW72 pad 4: 3.3V -> NEOPIX_PWR
- SW73 pad 4: 3.3V -> NEOPIX_PWR
- SW74 pad 4: 3.3V -> NEOPIX_PWR
- SW75 pad 4: 3.3V -> NEOPIX_PWR
- SW76 pad 4: 3.3V -> NEOPIX_PWR
- SW77 pad 4: 3.3V -> NEOPIX_PWR
- SW78 pad 4: 3.3V -> NEOPIX_PWR
- SW79 pad 4: 3.3V -> NEOPIX_PWR
- SW8 pad 4: 3.3V -> NEOPIX_PWR
- SW80 pad 4: 3.3V -> NEOPIX_PWR
- SW81 pad 4: 3.3V -> NEOPIX_PWR
- SW82 pad 4: 3.3V -> NEOPIX_PWR
- SW83 pad 4: 3.3V -> NEOPIX_PWR
- SW9 pad 4: 3.3V -> NEOPIX_PWR
- U1 pad 11: 4 -> /VDIV
- U1 pad 12: /VDIV -> 4
- U1 pad 42: /LED2 -> NEOPIX_EN
- U1 pad 43: /LED1 -> NEOPIX
- U1 pad 49: NEOPIX -> /LED2
- U1 pad 50: 10 -> /LED1
Routing:
- net 3.3V: track 284.7 -> 58.5 mm, vias 84 -> 4
- net NEOPIX_PWR: track 0.00 -> 225.8 mm, vias 0 -> 80
- net VBUS: track 384.4 -> 395.8 mm, vias 12 -> 10
- net VBAT: track 306.3 -> 314.4 mm
- net /USBD+: track 60.3 -> 55.9 mm
- net /USBD-: track 60.3 -> 55.9 mm
- net NEOPIX_EN: track 0.00 -> 1.17 mm, vias 0 -> 1
- net 10: track 1.12 -> 0.00 mm, vias 1 -> 0

Commit message: Moved the battery charger circuit
Parts:
- added R16: 470R, Resistor_SMD:R_0603_1608Metric, B.Cu at (203.2, 137.9)
- moved R10 215.1 mm to (336.5, 109.2), turned to -90 degrees
- moved R9 213.5 mm to (336.5, 105.7), turned to -90 degrees
- moved C6 205.8 mm to (330.3, 114.8), turned to 0 degrees
- moved R4 201.6 mm to (327.6, 112.9), turned to -90 degrees
- moved U3 200.9 mm to (330.3, 110.8), turned to -90 degrees
- moved R12 198.4 mm to (327.7, 110.2), turned to 90 degrees
- moved C9 195.8 mm to (330.3, 106.6), turned to 0 degrees
- moved J6 184.5 mm to (330.8, 100.2), turned to 180 degrees
- moved Q4 28.9 mm to (161.9, 152.5), turned to 0 degrees
- moved R14 27.5 mm to (154.6, 152.5), turned to -90 degrees
- moved Q2 27.3 mm to (157.5, 152.5), turned to 0 degrees
- moved R15 24.0 mm to (161.9, 155.1), turned to 0 degrees
- moved R13 21.5 mm to (157.4, 155.3)
- moved J5 19.0 mm to (151.3, 156.4)
- moved J2 16.5 mm to (140.0, 156.4)
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Connections:
- U1 pad 43: NEOPIX -> Net-(U1A-P0.22)
Routing:
- net VBUS: track 395.8 -> 85.9 mm, vias 10 -> 9
- net VBAT: track 314.4 -> 14.9 mm, vias 15 -> 11
- net NEOPIX: track 114.0 -> 283.4 mm
- net NEOPIX_EN: track 1.17 -> 58.1 mm, vias 1 -> 2
- net Net-(D85-K): track 48.9 -> 1.01 mm, vias 2 -> 1
- net /LED2: track 43.8 -> 1.15 mm, vias 2 -> 1
- net /LED1: track 38.5 -> 1.12 mm, vias 2 -> 1
- net Net-(D84-R): track 25.4 -> 1.48 mm, vias 2 -> 0
- net Net-(D84-G): track 17.3 -> 1.48 mm, vias 2 -> 0
- net Net-(Q2-D): track 0.00 -> 4.60 mm
- net NEOPIX_PWR: track 225.8 -> 229.7 mm, vias 80 -> 86
- net Net-(Q2-G): track 0.00 -> 3.89 mm
- net Net-(U1A-P0.22): track 0.00 -> 3.22 mm
- net GND: track 11.1 -> 8.41 mm, vias 444 -> 437
- net Net-(Q1A-B1): track 4.09 -> 1.75 mm
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- added copper zone on In1.Cu, net NEOPIX_PWR
- removed copper zone on In1.Cu, net 3.3V
Other:
- board size 330.2 x 118.6 mm -> 330.2 x 118.7 mm

Commit message: Worked on the layout, not sure its good
Parts:
- moved J2 74.3 mm to (213.5, 145.7)
- moved J5 62.7 mm to (213.5, 148.9)
- moved J10 2.90 mm to (369.8, 151.3)
Routing:
- net VBAT: track 14.9 -> 324.8 mm
- net VBUS: track 85.9 -> 341.2 mm, vias 9 -> 11
- net /VDIV: track 2.97 -> 245.6 mm
- net Net-(SW73B-DO): track 185.6 -> 374.4 mm
- net Col15: track 111.3 -> 250.5 mm, vias 6 -> 7
- net Col14: track 114.4 -> 238.0 mm, vias 7 -> 8
- net Col1: track 140.1 -> 248.0 mm
- net Col2: track 144.5 -> 251.4 mm
- net Col0: track 149.1 -> 255.9 mm
- net Col13: track 128.3 -> 214.7 mm, vias 8 -> 9
- net Col3: track 111.1 -> 194.2 mm
- net Row5: track 190.0 -> 271.3 mm
- net Row4: track 333.8 -> 412.7 mm
- net Row1: track 439.6 -> 518.3 mm
- net Row2: track 402.2 -> 480.7 mm
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
Commit message: small changes in the right direction
Parts:
- moved D1 16.6 mm to (62.7, 53.4), turned to -90 degrees
- moved D33 16.6 mm to (91.4, 96.4), turned to -90 degrees
- moved D34 16.6 mm to (110.4, 96.4), turned to -90 degrees
- moved D35 16.6 mm to (129.5, 96.4), turned to -90 degrees
- moved D43 16.6 mm to (281.9, 96.4), turned to -90 degrees
- moved D58 16.6 mm to (267.6, 115.4), turned to -90 degrees
- moved D45 16.5 mm to (324.7, 96.4), turned to -90 degrees
- moved D46 16.5 mm to (353.2, 96.4), turned to -90 degrees
- moved D32 16.5 mm to (67.5, 96.4), turned to -90 degrees
- moved D16 16.5 mm to (62.7, 77.3), turned to -90 degrees
- moved D79 16.5 mm to (279.5, 153.5), turned to -90 degrees
- moved D26 16.5 mm to (253.3, 77.3), turned to -90 degrees
- moved D37 16.5 mm to (167.4, 96.4), turned to -90 degrees
- moved D38 16.5 mm to (186.5, 96.4), turned to -90 degrees
- moved D40 16.5 mm to (224.6, 96.4), turned to -90 degrees
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Connections:
- D1 pad 1: Col0 -> Net-(D1-K)
- D1 pad 2: Net-(D1-A) -> Row0
- D10 pad 1: Col10 -> Net-(D10-K)
- D10 pad 2: Net-(D10-A) -> Row0
- D11 pad 1: Col11 -> Net-(D11-K)
- D11 pad 2: Net-(D11-A) -> Row0
- D12 pad 1: Col12 -> Net-(D12-K)
- D12 pad 2: Net-(D12-A) -> Row0
- D13 pad 1: Col13 -> Net-(D13-K)
- D13 pad 2: Net-(D13-A) -> Row0
- D14 pad 1: Col14 -> Net-(D14-K)
- D14 pad 2: Net-(D14-A) -> Row0
- D15 pad 1: Col15 -> Net-(D15-K)
- D15 pad 2: Net-(D15-A) -> Row0
- D16 pad 1: Col0 -> Net-(D16-K)
- D16 pad 2: Net-(D16-A) -> Row1
- D17 pad 1: Col1 -> Net-(D17-K)
- D17 pad 2: Net-(D17-A) -> Row1
- D18 pad 1: Col2 -> Net-(D18-K)
- D18 pad 2: Net-(D18-A) -> Row1
- D19 pad 1: Col3 -> Net-(D19-K)
- D19 pad 2: Net-(D19-A) -> Row1
- D2 pad 1: Col1 -> Net-(D2-K)
- D2 pad 2: Net-(D2-A) -> Row0
- D20 pad 1: Col4 -> Net-(D20-K)
- D20 pad 2: Net-(D20-A) -> Row1
- D21 pad 1: Col5 -> Net-(D21-K)
- D21 pad 2: Net-(D21-A) -> Row1
- D22 pad 1: Col6 -> Net-(D22-K)
- D22 pad 2: Net-(D22-A) -> Row1
- D23 pad 1: Col7 -> Net-(D23-K)
- D23 pad 2: Net-(D23-A) -> Row1
- D24 pad 1: Col8 -> Net-(D24-K)
- D24 pad 2: Net-(D24-A) -> Row1
- D25 pad 1: Col9 -> Net-(D25-K)
- D25 pad 2: Net-(D25-A) -> Row1
- D26 pad 1: Col10 -> Net-(D26-K)
- D26 pad 2: Net-(D26-A) -> Row1
- D27 pad 1: Col11 -> Net-(D27-K)
- D27 pad 2: Net-(D27-A) -> Row1
- D28 pad 1: Col12 -> Net-(D28-K)
- D28 pad 2: Net-(D28-A) -> Row1
- D29 pad 1: Col13 -> Net-(D29-K)
- D29 pad 2: Net-(D29-A) -> Row1
- D3 pad 1: Col2 -> Net-(D3-K)
- D3 pad 2: Net-(D3-A) -> Row0
- D30 pad 1: Col14 -> Net-(D30-K)
- D30 pad 2: Net-(D30-A) -> Row1
- D31 pad 1: Col15 -> Net-(D31-K)
- D31 pad 2: Net-(D31-A) -> Row1
- D32 pad 1: Col0 -> Net-(D32-K)
- D32 pad 2: Net-(D32-A) -> Row2
- D33 pad 1: Col1 -> Net-(D33-K)
- D33 pad 2: Net-(D33-A) -> Row2
- D34 pad 1: Col2 -> Net-(D34-K)
- D34 pad 2: Net-(D34-A) -> Row2
- D35 pad 1: Col3 -> Net-(D35-K)
- D35 pad 2: Net-(D35-A) -> Row2
- D36 pad 1: Col4 -> Net-(D36-K)
- D36 pad 2: Net-(D36-A) -> Row2
- D37 pad 1: Col5 -> Net-(D37-K)
- D37 pad 2: Net-(D37-A) -> Row2
- D38 pad 1: Col6 -> Net-(D38-K)
- D38 pad 2: Net-(D38-A) -> Row2
- D39 pad 1: Col7 -> Net-(D39-K)
- D39 pad 2: Net-(D39-A) -> Row2
- D4 pad 1: Col3 -> Net-(D4-K)
- D4 pad 2: Net-(D4-A) -> Row0
- D40 pad 1: Col8 -> Net-(D40-K)
- D40 pad 2: Net-(D40-A) -> Row2
- D41 pad 1: Col9 -> Net-(D41-K)
- D41 pad 2: Net-(D41-A) -> Row2
- D42 pad 1: Col10 -> Net-(D42-K)
- D42 pad 2: Net-(D42-A) -> Row2
- D43 pad 1: Col11 -> Net-(D43-K)
- D43 pad 2: Net-(D43-A) -> Row2
- D44 pad 1: Col12 -> Net-(D44-K)
- D44 pad 2: Net-(D44-A) -> Row2
- D45 pad 1: Col13 -> Net-(D45-K)
- D45 pad 2: Net-(D45-A) -> Row2
- D46 pad 1: Col14 -> Net-(D46-K)
- D46 pad 2: Net-(D46-A) -> Row2
- D47 pad 1: Col15 -> Net-(D47-K)
- D47 pad 2: Net-(D47-A) -> Row2
- D48 pad 1: Col0 -> Net-(D48-K)
- D48 pad 2: Net-(D48-A) -> Row3
- D49 pad 1: Col1 -> Net-(D49-K)
- D49 pad 2: Net-(D49-A) -> Row3
- D5 pad 1: Col4 -> Net-(D5-K)
- D5 pad 2: Net-(D5-A) -> Row0
- D50 pad 1: Col2 -> Net-(D50-K)
- D50 pad 2: Net-(D50-A) -> Row3
- D51 pad 1: Col3 -> Net-(D51-K)
- D51 pad 2: Net-(D51-A) -> Row3
- D52 pad 1: Col4 -> Net-(D52-K)
- D52 pad 2: Net-(D52-A) -> Row3
- D53 pad 1: Col5 -> Net-(D53-K)
- D53 pad 2: Net-(D53-A) -> Row3
- D54 pad 1: Col6 -> Net-(D54-K)
- D54 pad 2: Net-(D54-A) -> Row3
- D55 pad 1: Col7 -> Net-(D55-K)
- D55 pad 2: Net-(D55-A) -> Row3
- D56 pad 1: Col8 -> Net-(D56-K)
- D56 pad 2: Net-(D56-A) -> Row3
- D57 pad 1: Col9 -> Net-(D57-K)
- D57 pad 2: Net-(D57-A) -> Row3
- D58 pad 1: Col10 -> Net-(D58-K)
- D58 pad 2: Net-(D58-A) -> Row3
- D59 pad 1: Col11 -> Net-(D59-K)
- D59 pad 2: Net-(D59-A) -> Row3
- D6 pad 1: Col6 -> Net-(D6-K)
- D6 pad 2: Net-(D6-A) -> Row0
- D60 pad 1: Col13 -> Net-(D60-K)
- D60 pad 2: Net-(D60-A) -> Row3
- D61 pad 1: Col0 -> Net-(D61-K)
- D61 pad 2: Net-(D61-A) -> Row4
- D62 pad 1: Col1 -> Net-(D62-K)
- D62 pad 2: Net-(D62-A) -> Row4
- D63 pad 1: Col2 -> Net-(D63-K)
- D63 pad 2: Net-(D63-A) -> Row4
- D64 pad 1: Col3 -> Net-(D64-K)
- D64 pad 2: Net-(D64-A) -> Row4
- D65 pad 1: Col4 -> Net-(D65-K)
- D65 pad 2: Net-(D65-A) -> Row4
- D66 pad 1: Col5 -> Net-(D66-K)
- D66 pad 2: Net-(D66-A) -> Row4
- D67 pad 1: Col6 -> Net-(D67-K)
- D67 pad 2: Net-(D67-A) -> Row4
- D68 pad 1: Col7 -> Net-(D68-K)
- D68 pad 2: Net-(D68-A) -> Row4
- D69 pad 1: Col8 -> Net-(D69-K)
- D69 pad 2: Net-(D69-A) -> Row4
- D7 pad 1: Col7 -> Net-(D7-K)
- D7 pad 2: Net-(D7-A) -> Row0
- D70 pad 1: Col9 -> Net-(D70-K)
- D70 pad 2: Net-(D70-A) -> Row4
- D71 pad 1: Col10 -> Net-(D71-K)
- D71 pad 2: Net-(D71-A) -> Row4
- D72 pad 1: Col13 -> Net-(D72-K)
- D72 pad 2: Net-(D72-A) -> Row4
- D73 pad 1: Col14 -> Net-(D73-K)
- D73 pad 2: Net-(D73-A) -> Row4
- D74 pad 1: Col0 -> Net-(D74-K)
- D74 pad 2: Net-(D74-A) -> Row5
- D75 pad 1: Col1 -> Net-(D75-K)
- D75 pad 2: Net-(D75-A) -> Row5
- D76 pad 1: Col2 -> Net-(D76-K)
- D76 pad 2: Net-(D76-A) -> Row5
- D77 pad 1: Col5 -> Net-(D77-K)
- D77 pad 2: Net-(D77-A) -> Row5
- D78 pad 1: Col9 -> Net-(D78-K)
- D78 pad 2: Net-(D78-A) -> Row5
- D79 pad 1: Col10 -> Net-(D79-K)
- D79 pad 2: Net-(D79-A) -> Row5
- D8 pad 1: Col8 -> Net-(D8-K)
- D8 pad 2: Net-(D8-A) -> Row0
- D80 pad 1: Col12 -> Net-(D80-K)
- D80 pad 2: Net-(D80-A) -> Row5
- D81 pad 1: Col13 -> Net-(D81-K)
- D81 pad 2: Net-(D81-A) -> Row5
- D82 pad 1: Col14 -> Net-(D82-K)
- D82 pad 2: Net-(D82-A) -> Row5
- D83 pad 1: Col15 -> Net-(D83-K)
- D83 pad 2: Net-(D83-A) -> Row5
- D9 pad 1: Col9 -> Net-(D9-K)
- D9 pad 2: Net-(D9-A) -> Row0
- SW1 pad 1: Row0 -> Net-(D1-K)
- SW1 pad 2: Net-(D1-A) -> Col0
- SW10 pad 1: Row0 -> Net-(D10-K)
- SW10 pad 2: Net-(D10-A) -> Col10
- SW11 pad 1: Row0 -> Net-(D11-K)
- SW11 pad 2: Net-(D11-A) -> Col11
- SW12 pad 1: Row0 -> Net-(D12-K)
- SW12 pad 2: Net-(D12-A) -> Col12
- SW13 pad 1: Row0 -> Net-(D13-K)
- SW13 pad 2: Net-(D13-A) -> Col13
- SW14 pad 1: Row0 -> Net-(D14-K)
- SW14 pad 2: Net-(D14-A) -> Col14
- SW15 pad 1: Row0 -> Net-(D15-K)
- SW15 pad 2: Net-(D15-A) -> Col15
- SW16 pad 1: Row1 -> Net-(D16-K)
- SW16 pad 2: Net-(D16-A) -> Col0
- SW17 pad 1: Row1 -> Net-(D17-K)
- SW17 pad 2: Net-(D17-A) -> Col1
- SW18 pad 1: Row1 -> Net-(D18-K)
- SW18 pad 2: Net-(D18-A) -> Col2
- SW19 pad 1: Row1 -> Net-(D19-K)
- SW19 pad 2: Net-(D19-A) -> Col3
- SW2 pad 1: Row0 -> Net-(D2-K)
- SW2 pad 2: Net-(D2-A) -> Col1
- SW20 pad 1: Row1 -> Net-(D20-K)
- SW20 pad 2: Net-(D20-A) -> Col4
- SW21 pad 1: Row1 -> Net-(D21-K)
- SW21 pad 2: Net-(D21-A) -> Col5
- SW22 pad 1: Row1 -> Net-(D22-K)
- SW22 pad 2: Net-(D22-A) -> Col6
- SW23 pad 1: Row1 -> Net-(D23-K)
- SW23 pad 2: Net-(D23-A) -> Col7
- SW24 pad 1: Row1 -> Net-(D24-K)
- SW24 pad 2: Net-(D24-A) -> Col8
- SW25 pad 1: Row1 -> Net-(D25-K)
- SW25 pad 2: Net-(D25-A) -> Col9
- SW26 pad 1: Row1 -> Net-(D26-K)
- SW26 pad 2: Net-(D26-A) -> Col10
- SW27 pad 1: Row1 -> Net-(D27-K)
- SW27 pad 2: Net-(D27-A) -> Col11
- SW28 pad 1: Row1 -> Net-(D28-K)
- SW28 pad 2: Net-(D28-A) -> Col12
- SW29 pad 1: Row1 -> Net-(D29-K)
- SW29 pad 2: Net-(D29-A) -> Col13
- SW3 pad 1: Row0 -> Net-(D3-K)
- SW3 pad 2: Net-(D3-A) -> Col2
- SW30 pad 1: Row1 -> Net-(D30-K)
- SW30 pad 2: Net-(D30-A) -> Col14
- SW31 pad 1: Row1 -> Net-(D31-K)
- SW31 pad 2: Net-(D31-A) -> Col15
- SW32 pad 1: Row2 -> Net-(D32-K)
- SW32 pad 2: Net-(D32-A) -> Col0
- SW33 pad 1: Row2 -> Net-(D33-K)
- SW33 pad 2: Net-(D33-A) -> Col1
- SW34 pad 1: Row2 -> Net-(D34-K)
- SW34 pad 2: Net-(D34-A) -> Col2
- SW35 pad 1: Row2 -> Net-(D35-K)
- SW35 pad 2: Net-(D35-A) -> Col3
- SW36 pad 1: Row2 -> Net-(D36-K)
- SW36 pad 2: Net-(D36-A) -> Col4
- SW37 pad 1: Row2 -> Net-(D37-K)
- SW37 pad 2: Net-(D37-A) -> Col5
- SW38 pad 1: Row2 -> Net-(D38-K)
- SW38 pad 2: Net-(D38-A) -> Col6
- SW39 pad 1: Row2 -> Net-(D39-K)
- SW39 pad 2: Net-(D39-A) -> Col7
- SW4 pad 1: Row0 -> Net-(D4-K)
- SW4 pad 2: Net-(D4-A) -> Col3
- SW40 pad 1: Row2 -> Net-(D40-K)
- SW40 pad 2: Net-(D40-A) -> Col8
- SW41 pad 1: Row2 -> Net-(D41-K)
- SW41 pad 2: Net-(D41-A) -> Col9
- SW42 pad 1: Row2 -> Net-(D42-K)
- SW42 pad 2: Net-(D42-A) -> Col10
- SW43 pad 1: Row2 -> Net-(D43-K)
- SW43 pad 2: Net-(D43-A) -> Col11
- SW44 pad 1: Row2 -> Net-(D44-K)
- SW44 pad 2: Net-(D44-A) -> Col12
- SW45 pad 1: Row2 -> Net-(D45-K)
- SW45 pad 2: Net-(D45-A) -> Col13
- SW46 pad 1: Row2 -> Net-(D46-K)
- SW46 pad 2: Net-(D46-A) -> Col14
- SW47 pad 1: Row2 -> Net-(D47-K)
- SW47 pad 2: Net-(D47-A) -> Col15
- SW48 pad 1: Row3 -> Net-(D48-K)
- SW48 pad 2: Net-(D48-A) -> Col0
- SW49 pad 1: Row3 -> Net-(D49-K)
- SW49 pad 2: Net-(D49-A) -> Col1
- SW5 pad 1: Row0 -> Net-(D5-K)
- SW5 pad 2: Net-(D5-A) -> Col4
- SW50 pad 1: Row3 -> Net-(D50-K)
- SW50 pad 2: Net-(D50-A) -> Col2
- SW51 pad 1: Row3 -> Net-(D51-K)
- SW51 pad 2: Net-(D51-A) -> Col3
- SW52 pad 1: Row3 -> Net-(D52-K)
- SW52 pad 2: Net-(D52-A) -> Col4
- SW53 pad 1: Row3 -> Net-(D53-K)
- SW53 pad 2: Net-(D53-A) -> Col5
- SW54 pad 1: Row3 -> Net-(D54-K)
- SW54 pad 2: Net-(D54-A) -> Col6
- SW55 pad 1: Row3 -> Net-(D55-K)
- SW55 pad 2: Net-(D55-A) -> Col7
- SW56 pad 1: Row3 -> Net-(D56-K)
- SW56 pad 2: Net-(D56-A) -> Col8
- SW57 pad 1: Row3 -> Net-(D57-K)
- SW57 pad 2: Net-(D57-A) -> Col9
- SW58 pad 1: Row3 -> Net-(D58-K)
- SW58 pad 2: Net-(D58-A) -> Col10
- SW59 pad 1: Row3 -> Net-(D59-K)
- SW59 pad 2: Net-(D59-A) -> Col11
- SW6 pad 1: Row0 -> Net-(D6-K)
- SW6 pad 2: Net-(D6-A) -> Col6
- SW60 pad 1: Row3 -> Net-(D60-K)
- SW60 pad 2: Net-(D60-A) -> Col13
- SW61 pad 1: Row4 -> Net-(D61-K)
- SW61 pad 2: Net-(D61-A) -> Col0
- SW62 pad 1: Row4 -> Net-(D62-K)
- SW62 pad 2: Net-(D62-A) -> Col1
- SW63 pad 1: Row4 -> Net-(D63-K)
- SW63 pad 2: Net-(D63-A) -> Col2
- SW64 pad 1: Row4 -> Net-(D64-K)
- SW64 pad 2: Net-(D64-A) -> Col3
- SW65 pad 1: Row4 -> Net-(D65-K)
- SW65 pad 2: Net-(D65-A) -> Col4
- SW66 pad 1: Row4 -> Net-(D66-K)
- SW66 pad 2: Net-(D66-A) -> Col5
- SW67 pad 1: Row4 -> Net-(D67-K)
- SW67 pad 2: Net-(D67-A) -> Col6
- SW68 pad 1: Row4 -> Net-(D68-K)
- SW68 pad 2: Net-(D68-A) -> Col7
- SW69 pad 1: Row4 -> Net-(D69-K)
- SW69 pad 2: Net-(D69-A) -> Col8
- SW7 pad 1: Row0 -> Net-(D7-K)
- SW7 pad 2: Net-(D7-A) -> Col7
- SW70 pad 1: Row4 -> Net-(D70-K)
- SW70 pad 2: Net-(D70-A) -> Col9
- SW71 pad 1: Row4 -> Net-(D71-K)
- SW71 pad 2: Net-(D71-A) -> Col10
- SW72 pad 1: Row4 -> Net-(D72-K)
- SW72 pad 2: Net-(D72-A) -> Col13
- SW73 pad 1: Row4 -> Net-(D73-K)
- SW73 pad 2: Net-(D73-A) -> Col14
- SW74 pad 1: Row5 -> Net-(D74-K)
- SW74 pad 2: Net-(D74-A) -> Col0
- SW75 pad 1: Row5 -> Net-(D75-K)
- SW75 pad 2: Net-(D75-A) -> Col1
- SW76 pad 1: Row5 -> Net-(D76-K)
- SW76 pad 2: Net-(D76-A) -> Col2
- SW77 pad 1: Row5 -> Net-(D77-K)
- SW77 pad 2: Net-(D77-A) -> Col5
- SW78 pad 1: Row5 -> Net-(D78-K)
- SW78 pad 2: Net-(D78-A) -> Col9
- SW79 pad 1: Row5 -> Net-(D79-K)
- SW79 pad 2: Net-(D79-A) -> Col10
- SW8 pad 1: Row0 -> Net-(D8-K)
- SW8 pad 2: Net-(D8-A) -> Col8
- SW80 pad 1: Row5 -> Net-(D80-K)
- SW80 pad 2: Net-(D80-A) -> Col12
- SW81 pad 1: Row5 -> Net-(D81-K)
- SW81 pad 2: Net-(D81-A) -> Col13
- SW82 pad 1: Row5 -> Net-(D82-K)
- SW82 pad 2: Net-(D82-A) -> Col14
- SW83 pad 1: Row5 -> Net-(D83-K)
- SW83 pad 2: Net-(D83-A) -> Col15
- SW9 pad 1: Row0 -> Net-(D9-K)
- SW9 pad 2: Net-(D9-A) -> Col9
Routing:
- net Row1: track 518.3 -> 66.3 mm, vias 4 -> 1
- net Row2: track 480.7 -> 68.7 mm, vias 2 -> 1
- net Net-(SW73B-DO): track 374.4 -> 0.00 mm, vias 2 -> 0
- net Net-(SW31B-DO): track 350.5 -> 0.00 mm, vias 2 -> 0
- net Net-(SW15B-DO): track 359.4 -> 11.2 mm
- net Net-(SW47B-DO): track 338.8 -> 0.00 mm, vias 2 -> 0
- net Row4: track 412.7 -> 75.1 mm, vias 2 -> 1
- net Row3: track 392.6 -> 71.5 mm, vias 2 -> 1
- net Net-(SW60B-DO): track 298.0 -> 0.00 mm, vias 2 -> 0
- net VBAT: track 324.8 -> 43.2 mm
- net NEOPIX: track 276.3 -> 0.61 mm, vias 2 -> 0
- net VBUS: track 341.2 -> 97.7 mm
- net /VDIV: track 245.6 -> 14.0 mm
- net Row5: track 271.3 -> 79.5 mm, vias 4 -> 1
- net Row0: track 568.5 -> 388.7 mm, vias 4 -> 1
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