File: PCB/Every83_PCB.kicad_pcb (KiCad board)
At the start: 4 copper layers, 330.2 x 118.7 mm, 295 parts, among them J1 781710004, J10 Conn_01x01, J2 Conn_01x08_Socket, J5 Conn_01x08_Socket, J6 Conn_01x02_Pin, J7 Conn_02x03_Counter_Clockwise, Q1 MMDT2222A, Q2 2N7002, Q3 DMG2305, Q4 AO3401A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

Commit message: More work done. getting closer
Routing:
- net Row1: track 66.3 -> 582.1 mm
- net Row2: track 68.7 -> 554.0 mm
- net Row3: track 71.5 -> 461.6 mm
- net Row4: track 75.1 -> 459.8 mm
- net Row0: track 388.7 -> 607.9 mm
- net Net-(SW77B-DO): track 59.5 -> 4.44 mm
- net Row5: track 79.5 -> 60.6 mm
- net Net-(D52-K): track 5.06 -> 8.89 mm
- net Net-(D50-K): track 3.91 -> 7.74 mm
- net Net-(D49-K): track 3.96 -> 7.79 mm
- net Net-(D60-K): track 4.11 -> 7.94 mm
- net Net-(D56-K): track 3.91 -> 7.74 mm
- net Net-(D55-K): track 5.04 -> 8.87 mm
- net Net-(D53-K): track 5.04 -> 8.87 mm
- net Net-(D51-K): track 3.91 -> 7.74 mm
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
Commit message: Add files via upload
Parts:
- moved Q1 127.8 mm to (191.6, 170.4)
- moved R11 127.8 mm to (192.6, 173.2)
- moved R2 127.8 mm to (191.1, 167.0)
- moved R3 127.8 mm to (194.1, 167.0)
- moved R5 127.8 mm to (190.6, 173.2)
- moved J7 44.6 mm to (235.1, 147.8)
- moved R9 18.0 mm to (332.3, 123.3)
- moved R10 18.0 mm to (332.3, 126.8)
- moved C9 17.8 mm to (327.4, 124.2)
- moved U3 17.8 mm to (327.4, 128.4)
- moved R12 17.8 mm to (324.8, 127.7)
- moved C6 17.8 mm to (327.4, 132.3)
- moved J6 17.8 mm to (327.9, 117.7)
- moved R4 17.8 mm to (324.7, 130.4)
- moved Q4 16.1 mm to (145.8, 151.4)
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Routing:
- net Row5: track 60.6 -> 322.7 mm, vias 1 -> 0
- net NEOPIX_EN: track 67.8 -> 0.71 mm, vias 2 -> 1
- net VBUS: track 97.7 -> 34.8 mm
- net Row4: track 459.8 -> 508.1 mm, vias 1 -> 2
- net Row3: track 461.6 -> 495.2 mm, vias 1 -> 2
- net Col8: track 142.0 -> 115.2 mm
- net /SWDIO: track 26.9 -> 1.14 mm, vias 2 -> 1
- net /SWDCLK: track 23.7 -> 1.15 mm, vias 2 -> 1
- net /TXD: track 21.5 -> 0.00 mm, vias 2 -> 0
- net VBAT: track 43.2 -> 21.9 mm
- net /RXD: track 21.1 -> 0.00 mm, vias 2 -> 0
- net Row2: track 554.0 -> 574.0 mm, vias 1 -> 2
- net Col6: track 128.0 -> 115.2 mm
- net Col5: track 121.0 -> 109.3 mm
- net Col7: track 126.3 -> 115.2 mm
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
Commit message: Add files via upload
Routing:
- net Col15: track 116.8 -> 448.4 mm
- net Col14: track 121.2 -> 434.3 mm
- net Col13: track 148.9 -> 431.9 mm
- net Col12: track 129.6 -> 373.2 mm
- net Col11: track 92.6 -> 317.4 mm
- net Col10: track 143.4 -> 348.0 mm
- net Col9: track 139.4 -> 324.4 mm
- net Col8: track 115.2 -> 281.5 mm
- net Col7: track 115.2 -> 261.2 mm
- net Col6: track 115.2 -> 241.7 mm
- net Col5: track 109.3 -> 216.4 mm
- net Col4: track 119.2 -> 206.7 mm
- net Col3: track 119.2 -> 187.3 mm
- net Col2: track 147.1 -> 195.7 mm
- net Col1: track 149.0 -> 178.0 mm
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
Commit message: Add files via upload
Parts:
- moved R11 27.2 mm to (198.0, 146.5), turned to 180 degrees
- moved R5 26.4 mm to (198.1, 147.9), turned to 180 degrees
- moved Q1 23.2 mm to (195.4, 147.5)
- moved R3 20.4 mm to (192.9, 146.6), turned to 0 degrees
- moved R2 18.6 mm to (192.9, 148.4), turned to 0 degrees
- moved Q4 2.01 mm to (147.7, 150.7)
- moved R13 2.01 mm to (143.2, 153.5)
- moved R14 2.01 mm to (140.4, 150.7)
- moved R15 2.01 mm to (147.7, 153.4)
- moved Q2 2.01 mm to (143.4, 150.7)
Routing:
- net Col11: track 317.4 -> 579.2 mm, vias 5 -> 6
- net Col9: track 324.4 -> 585.5 mm, vias 7 -> 8
- net Col10: track 348.0 -> 608.8 mm, vias 7 -> 8
- net Col12: track 373.2 -> 632.4 mm, vias 5 -> 6
- net Col8: track 281.5 -> 534.4 mm, vias 6 -> 7
- net Col7: track 261.2 -> 513.1 mm, vias 6 -> 7
- net Col6: track 241.7 -> 491.8 mm, vias 6 -> 7
- net Col5: track 216.4 -> 465.1 mm, vias 6 -> 7
- net Col15: track 448.4 -> 693.2 mm, vias 5 -> 6
- net Col14: track 434.3 -> 679.0 mm, vias 6 -> 7
- net Col13: track 431.9 -> 676.3 mm, vias 7 -> 8
- net Col4: track 206.7 -> 268.6 mm, vias 6 -> 7
- net Col3: track 187.3 -> 248.7 mm, vias 6 -> 7
- net Col2: track 195.7 -> 256.7 mm, vias 7 -> 8
- net Col1: track 178.0 -> 238.7 mm, vias 7 -> 8
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